File: Poto-Rev2/Poto-Rev2.kicad_pcb (KiCad board)
At the start: 2 copper layers, 18 x 16.5 mm, 14 parts, among them J1 TYPE-C-31-M12_13, J2 SM04B-SRSS-TB(LF)(SN), U1 TPD4E05U06DQAR

Commit message: Big Chungus Update
Almost Everything Done
Parts:
- removed the MH3 at (68.0, 71.0)
- added C1: 0.1uF, Capacitor_SMD:C_0402_1005Metric_Pad0.74x0.62mm_HandSolder, B.Cu at (333.3, 102.6)
- added C2: 0.1uF, Capacitor_SMD:C_0402_1005Metric_Pad0.74x0.62mm_HandSolder, B.Cu at (328.7, 92.3)
- added C3: 0.1uF, Capacitor_SMD:C_0402_1005Metric_Pad0.74x0.62mm_HandSolder, B.Cu at (325.8, 99.8)
- added C4: 0.1uF, Capacitor_SMD:C_0402_1005Metric_Pad0.74x0.62mm_HandSolder, B.Cu at (334.1, 92.1)
- added C5: 10pF, Capacitor_SMD:C_0402_1005Metric_Pad0.74x0.62mm_HandSolder, B.Cu at (318.3, 97.5)
- added C6: 10pF, Capacitor_SMD:C_0402_1005Metric_Pad0.74x0.62mm_HandSolder, B.Cu at (318.4, 103.1)
- added C7: 0.1uF, Capacitor_SMD:C_0402_1005Metric_Pad0.74x0.62mm_HandSolder, B.Cu at (344.0, 101.0)
- added C8: 1uF, Capacitor_SMD:C_0402_1005Metric_Pad0.74x0.62mm_HandSolder, B.Cu at (337.9, 99.3)
- added D10: D_Small, Diode_SMD:D_SOD-123, B.Cu at (77.8, 169.1)
- added D100: D_Small, Diode_SMD:D_SOD-123, B.Cu at (363.5, 169.1)
- added D101: D_Small, Diode_SMD:D_SOD-123, B.Cu at (363.5, 188.1)
- added D102: D_Small, Diode_SMD:D_SOD-123, B.Cu at (363.5, 207.2)
- added D103: D_Small, Diode_SMD:D_SOD-123, B.Cu at (363.5, 226.2)
- added D11: D_Small, Diode_SMD:D_SOD-123, B.Cu at (77.8, 188.1)
- added D12: D_Small, Diode_SMD:D_SOD-123, B.Cu at (77.8, 207.2)
- added D13: D_Small, Diode_SMD:D_SOD-123, B.Cu at (77.8, 226.2)
- added D14: D_Small, Diode_SMD:D_SOD-123, B.Cu at (96.8, 131.0)
- added D15: D_Small, Diode_SMD:D_SOD-123, B.Cu at (96.8, 150.0)
- added D16: D_Small, Diode_SMD:D_SOD-123, B.Cu at (96.8, 169.1)
- added D17: D_Small, Diode_SMD:D_SOD-123, B.Cu at (96.8, 188.1)
- added D18: D_Small, Diode_SMD:D_SOD-123, B.Cu at (96.8, 207.2)
- added D19: D_Small, Diode_SMD:D_SOD-123, B.Cu at (96.8, 226.3)
- added D2: D_Small, Diode_SMD:D_SOD-123, B.Cu at (57.1, 131.0)
- added D20: D_Small, Diode_SMD:D_SOD-123, B.Cu at (115.9, 131.0)
- added D21: D_Small, Diode_SMD:D_SOD-123, B.Cu at (115.9, 150.0)
- added D22: D_Small, Diode_SMD:D_SOD-123, B.Cu at (115.9, 169.1)
- added D23: D_Small, Diode_SMD:D_SOD-123, B.Cu at (115.9, 188.1)
- added D24: D_Small, Diode_SMD:D_SOD-123, B.Cu at (115.9, 207.2)
- added D25: D_Small, Diode_SMD:D_SOD-123, B.Cu at (115.9, 226.2)
- added D26: D_Small, Diode_SMD:D_SOD-123, B.Cu at (134.9, 131.0)
- added D27: D_Small, Diode_SMD:D_SOD-123, B.Cu at (134.9, 150.0)
- added D28: D_Small, Diode_SMD:D_SOD-123, B.Cu at (134.9, 169.1)
- added D29: D_Small, Diode_SMD:D_SOD-123, B.Cu at (134.9, 188.1)
- added D3: D_Small, Diode_SMD:D_SOD-123, B.Cu at (58.7, 150.0)
- added D30: D_Small, Diode_SMD:D_SOD-123, B.Cu at (134.9, 207.2)
- added D31: D_Small, Diode_SMD:D_SOD-123, B.Cu at (134.9, 226.2)
- added D32: D_Small, Diode_SMD:D_SOD-123, B.Cu at (152.4, 131.0)
- added D33: D_Small, Diode_SMD:D_SOD-123, B.Cu at (154.0, 150.0)
- added D34: D_Small, Diode_SMD:D_SOD-123, B.Cu at (152.4, 169.1)
- added D35: D_Small, Diode_SMD:D_SOD-123, B.Cu at (154.0, 188.1)
- added D36: D_Small, Diode_SMD:D_SOD-123, B.Cu at (152.4, 207.2)
- added D37: D_Small, Diode_SMD:D_SOD-123, B.Cu at (154.0, 226.2)
- added D38: D_Small, Diode_SMD:D_SOD-123, B.Cu at (171.4, 131.0)
- added D39: D_Small, Diode_SMD:D_SOD-123, B.Cu at (173.0, 150.0)
- added D4: D_Small, Diode_SMD:D_SOD-123, B.Cu at (57.1, 169.1)
- added D40: D_Small, Diode_SMD:D_SOD-123, B.Cu at (171.4, 169.1)
- added D41: D_Small, Diode_SMD:D_SOD-123, B.Cu at (173.0, 188.1)
- added D42: D_Small, Diode_SMD:D_SOD-123, B.Cu at (171.4, 207.2)
- added D43: D_Small, Diode_SMD:D_SOD-123, B.Cu at (173.0, 226.3)
- added D44: D_Small, Diode_SMD:D_SOD-123, B.Cu at (192.1, 131.0)
- added D45: D_Small, Diode_SMD:D_SOD-123, B.Cu at (192.1, 150.0)
- added D46: D_Small, Diode_SMD:D_SOD-123, B.Cu at (192.1, 169.1)
- added D47: D_Small, Diode_SMD:D_SOD-123, B.Cu at (192.1, 188.1)
- added D48: D_Small, Diode_SMD:D_SOD-123, B.Cu at (192.1, 207.2)
- added D49: D_Small, Diode_SMD:D_SOD-123, B.Cu at (192.1, 226.2)
- added D5: D_Small, Diode_SMD:D_SOD-123, B.Cu at (58.7, 188.1)
- added D50: D_Small, Diode_SMD:D_SOD-123, B.Cu at (211.1, 131.0)
- added D51: D_Small, Diode_SMD:D_SOD-123, B.Cu at (211.1, 150.0)
- added D52: D_Small, Diode_SMD:D_SOD-123, B.Cu at (211.1, 169.1)
- added D53: D_Small, Diode_SMD:D_SOD-123, B.Cu at (211.1, 188.1)
- added D54: D_Small, Diode_SMD:D_SOD-123, B.Cu at (211.1, 207.2)
- added D55: D_Small, Diode_SMD:D_SOD-123, B.Cu at (211.1, 226.3)
- added D56: D_Small, Diode_SMD:D_SOD-123, B.Cu at (230.2, 131.0)
- added D57: D_Small, Diode_SMD:D_SOD-123, B.Cu at (230.2, 150.0)
- added D58: D_Small, Diode_SMD:D_SOD-123, B.Cu at (230.2, 169.1)
- added D59: D_Small, Diode_SMD:D_SOD-123, B.Cu at (230.2, 188.1)
- added D6: D_Small, Diode_SMD:D_SOD-123, B.Cu at (57.1, 207.2)
- added D60: D_Small, Diode_SMD:D_SOD-123, B.Cu at (230.2, 207.2)
- added D61: D_Small, Diode_SMD:D_SOD-123, B.Cu at (230.2, 226.2)
- added D62: D_Small, Diode_SMD:D_SOD-123, B.Cu at (249.2, 131.0)
- added D63: D_Small, Diode_SMD:D_SOD-123, B.Cu at (249.2, 150.0)
- added D64: D_Small, Diode_SMD:D_SOD-123, B.Cu at (249.2, 169.1)
- added D65: D_Small, Diode_SMD:D_SOD-123, B.Cu at (249.2, 188.1)
- added D66: D_Small, Diode_SMD:D_SOD-123, B.Cu at (249.2, 207.2)
- added D67: D_Small, Diode_SMD:D_SOD-123, B.Cu at (249.2, 226.2)
- added D68: D_Small, Diode_SMD:D_SOD-123, B.Cu at (266.7, 131.0)
- added D69: D_Small, Diode_SMD:D_SOD-123, B.Cu at (268.3, 150.0)
- added D7: D_Small, Diode_SMD:D_SOD-123, B.Cu at (58.7, 226.2)
- added D70: D_Small, Diode_SMD:D_SOD-123, B.Cu at (266.7, 169.1)
- added D71: D_Small, Diode_SMD:D_SOD-123, B.Cu at (268.3, 188.1)
- added D72: D_Small, Diode_SMD:D_SOD-123, B.Cu at (266.7, 207.2)
- added D73: D_Small, Diode_SMD:D_SOD-123, B.Cu at (268.3, 226.2)
- added D74: D_Small, Diode_SMD:D_SOD-123, B.Cu at (287.3, 131.0)
- added D75: D_Small, Diode_SMD:D_SOD-123, B.Cu at (287.3, 150.0)
- added D76: D_Small, Diode_SMD:D_SOD-123, B.Cu at (287.3, 169.1)
- added D77: D_Small, Diode_SMD:D_SOD-123, B.Cu at (287.3, 188.1)
- added D78: D_Small, Diode_SMD:D_SOD-123, B.Cu at (287.3, 207.2)
- added D79: D_Small, Diode_SMD:D_SOD-123, B.Cu at (287.3, 226.2)
- added D8: D_Small, Diode_SMD:D_SOD-123, B.Cu at (77.8, 131.0)
- added D80: D_Small, Diode_SMD:D_SOD-123, B.Cu at (304.8, 131.0)
- added D81: D_Small, Diode_SMD:D_SOD-123, B.Cu at (306.4, 150.0)
- added D82: D_Small, Diode_SMD:D_SOD-123, B.Cu at (304.8, 169.1)
- added D83: D_Small, Diode_SMD:D_SOD-123, B.Cu at (306.4, 188.1)
- added D84: D_Small, Diode_SMD:D_SOD-123, B.Cu at (304.8, 207.2)
- added D85: D_Small, Diode_SMD:D_SOD-123, B.Cu at (306.4, 226.2)
- added D86: D_Small, Diode_SMD:D_SOD-123, B.Cu at (325.4, 131.0)
- added D87: D_Small, Diode_SMD:D_SOD-123, B.Cu at (325.4, 150.0)
- added D88: D_Small, Diode_SMD:D_SOD-123, B.Cu at (325.4, 169.1)
- added D89: D_Small, Diode_SMD:D_SOD-123, B.Cu at (325.4, 188.1)
- added D9: D_Small, Diode_SMD:D_SOD-123, B.Cu at (77.8, 150.0)
- added D90: D_Small, Diode_SMD:D_SOD-123, B.Cu at (325.4, 207.2)
- added D91: D_Small, Diode_SMD:D_SOD-123, B.Cu at (325.4, 226.2)
- added D92: D_Small, Diode_SMD:D_SOD-123, B.Cu at (342.9, 131.0)
- added D93: D_Small, Diode_SMD:D_SOD-123, B.Cu at (344.5, 150.0)
- added D94: D_Small, Diode_SMD:D_SOD-123, B.Cu at (342.9, 169.1)
- added D95: D_Small, Diode_SMD:D_SOD-123, B.Cu at (344.5, 188.1)
- added D96: D_Small, Diode_SMD:D_SOD-123, B.Cu at (342.9, 207.2)
- added D97: D_Small, Diode_SMD:D_SOD-123, B.Cu at (344.5, 226.2)
- added D98: D_Small, Diode_SMD:D_SOD-123, B.Cu at (363.5, 131.0)
- added D99: D_Small, Diode_SMD:D_SOD-123, B.Cu at (363.5, 150.0)
- added G***: LOGO, Logo:poto, B.Cu at (347.1, 105.2)
- added J10: Conn_01x01, Connector_PinHeader_2.54mm:PinHeader_1x01_P2.54mm_Vertical, B.Cu at (336.7, 91.3)
- added J12: Conn_01x01, Connector_PinHeader_1.00mm:PinHeader_1x01_P1.00mm_Vertical, B.Cu at (326.5, 93.7)
- added J15: OLED, Connector_PinHeader_2.54mm:PinHeader_1x02_P2.54mm_Vertical, B.Cu at (325.1, 112.5)
- added J3: Conn_01x12, Connector_PinHeader_2.54mm:PinHeader_1x12_P2.54mm_Vertical, B.Cu at (341.8, 88.5)
- added J4: RGB, Connector_PinHeader_2.54mm:PinHeader_1x01_P2.54mm_Vertical, B.Cu at (301.1, 100.8)
- added J5: ENCODER, Connector_PinHeader_2.54mm:PinHeader_1x03_P2.54mm_Vertical, B.Cu at (301.1, 97.2)
- added J6: USB, random-keyboard-parts:JST-SR-4, B.Cu at (339.0, 95.6)
- added J7: Conn_01x12, Connector_PinHeader_2.54mm:PinHeader_1x12_P2.54mm_Vertical, B.Cu at (341.8, 105.3)
- added J8: Conn_01x01, Connector_PinHeader_2.54mm:PinHeader_1x01_P2.54mm_Vertical, B.Cu at (341.8, 101.7)
- added J9: Conn_01x05, Connector_PinHeader_2.54mm:PinHeader_1x05_P2.54mm_Vertical, B.Cu at (313.8, 91.6)
- added LED1: PWR, LED_SMD:LED_0201_0603Metric_Pad0.64x0.40mm_HandSolder, B.Cu at (342.8, 91.1)
- added LED2: BuiltIn, LED_SMD:LED_0201_0603Metric_Pad0.64x0.40mm_HandSolder, B.Cu at (319.8, 90.6)
- added MH3: Mount-M2, random-keyboard-parts:Generic-Mounthole, B.Cu at (308.0, 208.8)
- added MH3: Mount-M2, random-keyboard-parts:Generic-Mounthole, B.Cu at (174.6, 208.8)
- added MH3: Mount-M2, random-keyboard-parts:Generic-Mounthole, B.Cu at (174.6, 170.7)
- added MH3: Mount-M2, random-keyboard-parts:Generic-Mounthole, B.Cu at (174.6, 132.6)
- added MH3: Mount-M2, random-keyboard-parts:Generic-Mounthole, B.Cu at (155.6, 132.6)
- added MH3: Mount-M2, random-keyboard-parts:Generic-Mounthole, B.Cu at (155.6, 170.7)
- added MH3: Mount-M2, random-keyboard-parts:Generic-Mounthole, B.Cu at (155.6, 208.8)
- added MH3: Mount-M2, random-keyboard-parts:Generic-Mounthole, B.Cu at (60.3, 170.7)
- added MH3: Mount-M2, random-keyboard-parts:Generic-Mounthole, B.Cu at (60.3, 208.8)
- added MH3: Mount-M2, random-keyboard-parts:Generic-Mounthole, B.Cu at (60.3, 132.6)
- added MH3: Mount-M2, random-keyboard-parts:Generic-Mounthole, B.Cu at (363.1, 100.3)
- added MH3: Mount-M2, random-keyboard-parts:Generic-Mounthole, B.Cu at (308.0, 170.7)
- added MH3: Mount-M2, random-keyboard-parts:Generic-Mounthole, B.Cu at (308.0, 132.6)
- added MH3: Mount-M2, random-keyboard-parts:Generic-Mounthole, B.Cu at (346.1, 208.8)
- added MH3: Mount-M2, random-keyboard-parts:Generic-Mounthole, B.Cu at (346.1, 170.7)
- added MH3: Mount-M2, random-keyboard-parts:Generic-Mounthole, B.Cu at (346.1, 132.6)
- added MH3: Mount-M2, random-keyboard-parts:Generic-Mounthole, B.Cu at (269.9, 208.8)
- added MH3: Mount-M2, random-keyboard-parts:Generic-Mounthole, B.Cu at (269.9, 170.7)
- added MH3: Mount-M2, random-keyboard-parts:Generic-Mounthole, B.Cu at (269.9, 132.6)
- added MX1: MX-NoLED, MX_Only:MXOnly-1U-Hotswap-Antishear, F.Cu at (50.8, 126.2)
- added MX10: MX-NoLED, MX_Only:MXOnly-1U-Hotswap-Antishear, F.Cu at (69.8, 183.4)
- added MX100: MX-NoLED, MX_Only:MXOnly-1U-Hotswap-Antishear, F.Cu at (355.6, 183.4)
- added MX101: MX-NoLED, MX_Only:MXOnly-1U-Hotswap-Antishear, F.Cu at (355.6, 202.4)
- added MX102: MX-NoLED, MX_Only:MXOnly-1U-Hotswap-Antishear, F.Cu at (355.6, 221.5)
- added MX11: MX-NoLED, MX_Only:MXOnly-1U-Hotswap-Antishear, F.Cu at (69.8, 202.4)
- added MX12: MX-NoLED, MX_Only:MXOnly-1U-Hotswap-Antishear, F.Cu at (69.8, 221.5)
- added MX13: MX-NoLED, MX_Only:MXOnly-1U-Hotswap-Antishear, F.Cu at (88.9, 126.2)
- added MX14: MX-NoLED, MX_Only:MXOnly-1U-Hotswap-Antishear, F.Cu at (88.9, 145.3)
- added MX15: MX-NoLED, MX_Only:MXOnly-1U-Hotswap-Antishear, F.Cu at (88.9, 164.3)
- added MX16: MX-NoLED, MX_Only:MXOnly-1U-Hotswap-Antishear, F.Cu at (88.9, 183.4)
- added MX17: MX-NoLED, MX_Only:MXOnly-1U-Hotswap-Antishear, F.Cu at (88.9, 202.4)
- added MX18: MX-NoLED, MX_Only:MXOnly-1U-Hotswap-Antishear, F.Cu at (88.9, 221.5)
- added MX19: MX-NoLED, MX_Only:MXOnly-1U-Hotswap-Antishear, F.Cu at (108.0, 126.2)
- added MX2: MX-NoLED, MX_Only:MXOnly-1U-Hotswap-Antishear, F.Cu at (50.8, 145.3)
- added MX20: MX-NoLED, MX_Only:MXOnly-1U-Hotswap-Antishear, F.Cu at (108.0, 145.3)
- added MX21: MX-NoLED, MX_Only:MXOnly-1U-Hotswap-Antishear, F.Cu at (108.0, 164.3)
- added MX22: MX-NoLED, MX_Only:MXOnly-1U-Hotswap-Antishear, F.Cu at (108.0, 183.4)
- added MX23: MX-NoLED, MX_Only:MXOnly-1U-Hotswap-Antishear, F.Cu at (108.0, 202.4)
- added MX24: MX-NoLED, MX_Only:MXOnly-1U-Hotswap-Antishear, F.Cu at (108.0, 221.5)
- added MX25: MX-NoLED, MX_Only:MXOnly-1U-Hotswap-Antishear, F.Cu at (127.0, 126.2)
- added MX26: MX-NoLED, MX_Only:MXOnly-1U-Hotswap-Antishear, F.Cu at (127.0, 145.3)
- added MX27: MX-NoLED, MX_Only:MXOnly-1U-Hotswap-Antishear, F.Cu at (127.0, 164.3)
- added MX28: MX-NoLED, MX_Only:MXOnly-1U-Hotswap-Antishear, F.Cu at (127.0, 183.4)
- added MX29: MX-NoLED, MX_Only:MXOnly-1U-Hotswap-Antishear, F.Cu at (127.0, 202.4)
- added MX3: MX-NoLED, MX_Only:MXOnly-1U-Hotswap-Antishear, F.Cu at (50.8, 164.3)
- added MX30: MX-NoLED, MX_Only:MXOnly-1U-Hotswap-Antishear, F.Cu at (127.0, 221.5)
- added MX31: MX-NoLED, MX_Only:MXOnly-1U-Hotswap-Antishear, F.Cu at (146.1, 126.2)
- added MX32: MX-NoLED, MX_Only:MXOnly-1U-Hotswap-Antishear, F.Cu at (146.1, 145.3)
- added MX33: MX-NoLED, MX_Only:MXOnly-1U-Hotswap-Antishear, F.Cu at (146.1, 164.3)
- added MX34: MX-NoLED, MX_Only:MXOnly-1U-Hotswap-Antishear, F.Cu at (146.1, 183.4)
- added MX35: MX-NoLED, MX_Only:MXOnly-1U-Hotswap-Antishear, F.Cu at (146.1, 202.4)
- added MX36: MX-NoLED, MX_Only:MXOnly-1U-Hotswap-Antishear, F.Cu at (146.1, 221.5)
- added MX37: MX-NoLED, MX_Only:MXOnly-1U-Hotswap-Antishear, F.Cu at (165.1, 126.2)
- added MX38: MX-NoLED, MX_Only:MXOnly-1U-Hotswap-Antishear, F.Cu at (165.1, 145.3)
- added MX39: MX-NoLED, MX_Only:MXOnly-1U-Hotswap-Antishear, F.Cu at (165.1, 164.3)
- added MX4: MX-NoLED, MX_Only:MXOnly-1U-Hotswap-Antishear, F.Cu at (50.8, 183.4)
- added MX40: MX-NoLED, MX_Only:MXOnly-1U-Hotswap-Antishear, F.Cu at (165.1, 183.4)
- added MX41: MX-NoLED, MX_Only:MXOnly-1U-Hotswap-Antishear, F.Cu at (165.1, 202.4)
- added MX42: MX-NoLED, MX_Only:MXOnly-1U-Hotswap-Antishear, F.Cu at (165.1, 221.5)
- added MX43: MX-NoLED, MX_Only:MXOnly-1U-Hotswap-Antishear, F.Cu at (184.2, 126.2)
- added MX44: MX-NoLED, MX_Only:MXOnly-1U-Hotswap-Antishear, F.Cu at (184.2, 145.3)
- added MX45: MX-NoLED, MX_Only:MXOnly-1U-Hotswap-Antishear, F.Cu at (184.2, 164.3)
- added MX46: MX-NoLED, MX_Only:MXOnly-1U-Hotswap-Antishear, F.Cu at (184.2, 183.4)
- added MX47: MX-NoLED, MX_Only:MXOnly-1U-Hotswap-Antishear, F.Cu at (184.2, 202.4)
- added MX48: MX-NoLED, MX_Only:MXOnly-1U-Hotswap-Antishear, F.Cu at (184.2, 221.5)
- added MX49: MX-NoLED, MX_Only:MXOnly-1U-Hotswap-Antishear, F.Cu at (203.2, 126.2)
- added MX5: MX-NoLED, MX_Only:MXOnly-1U-Hotswap-Antishear, F.Cu at (50.8, 202.4)
- added MX50: MX-NoLED, MX_Only:MXOnly-1U-Hotswap-Antishear, F.Cu at (203.2, 145.3)
- added MX51: MX-NoLED, MX_Only:MXOnly-1U-Hotswap-Antishear, F.Cu at (203.2, 164.3)
- added MX52: MX-NoLED, MX_Only:MXOnly-1U-Hotswap-Antishear, F.Cu at (203.2, 183.4)
- added MX53: MX-NoLED, MX_Only:MXOnly-1U-Hotswap-Antishear, F.Cu at (203.2, 202.4)
- added MX54: MX-NoLED, MX_Only:MXOnly-1U-Hotswap-Antishear, F.Cu at (203.2, 221.5)
- added MX55: MX-NoLED, MX_Only:MXOnly-1U-Hotswap-Antishear, F.Cu at (222.2, 126.2)
- added MX56: MX-NoLED, MX_Only:MXOnly-1U-Hotswap-Antishear, F.Cu at (222.2, 145.3)
- added MX57: MX-NoLED, MX_Only:MXOnly-1U-Hotswap-Antishear, F.Cu at (222.2, 164.3)
- added MX58: MX-NoLED, MX_Only:MXOnly-1U-Hotswap-Antishear, F.Cu at (222.2, 183.4)
- added MX59: MX-NoLED, MX_Only:MXOnly-1U-Hotswap-Antishear, F.Cu at (222.2, 202.4)
- added MX6: MX-NoLED, MX_Only:MXOnly-1U-Hotswap-Antishear, F.Cu at (50.8, 221.5)
- added MX60: MX-NoLED, MX_Only:MXOnly-1U-Hotswap-Antishear, F.Cu at (222.2, 221.5)
- added MX61: MX-NoLED, MX_Only:MXOnly-1U-Hotswap-Antishear, F.Cu at (241.3, 126.2)
- added MX62: MX-NoLED, MX_Only:MXOnly-1U-Hotswap-Antishear, F.Cu at (241.3, 145.3)
- added MX63: MX-NoLED, MX_Only:MXOnly-1U-Hotswap-Antishear, F.Cu at (241.3, 164.3)
- added MX64: MX-NoLED, MX_Only:MXOnly-1U-Hotswap-Antishear, F.Cu at (241.3, 183.4)
- added MX65: MX-NoLED, MX_Only:MXOnly-1U-Hotswap-Antishear, F.Cu at (241.3, 202.4)
- added MX66: MX-NoLED, MX_Only:MXOnly-1U-Hotswap-Antishear, F.Cu at (241.3, 221.5)
- added MX67: MX-NoLED, MX_Only:MXOnly-1U-Hotswap-Antishear, F.Cu at (260.4, 126.2)
- added MX68: MX-NoLED, MX_Only:MXOnly-1U-Hotswap-Antishear, F.Cu at (260.4, 145.3)
- added MX69: MX-NoLED, MX_Only:MXOnly-1U-Hotswap-Antishear, F.Cu at (260.4, 164.3)
- added MX7: MX-NoLED, MX_Only:MXOnly-1U-Hotswap-Antishear, F.Cu at (69.8, 126.2)
- added MX70: MX-NoLED, MX_Only:MXOnly-1U-Hotswap-Antishear, F.Cu at (260.4, 183.4)
- added MX71: MX-NoLED, MX_Only:MXOnly-1U-Hotswap-Antishear, F.Cu at (260.4, 202.4)
- added MX72: MX-NoLED, MX_Only:MXOnly-1U-Hotswap-Antishear, F.Cu at (260.4, 221.5)
- added MX73: MX-NoLED, MX_Only:MXOnly-1U-Hotswap-Antishear, F.Cu at (279.4, 126.2)
- added MX74: MX-NoLED, MX_Only:MXOnly-1U-Hotswap-Antishear, F.Cu at (279.4, 145.3)
- added MX75: MX-NoLED, MX_Only:MXOnly-1U-Hotswap-Antishear, F.Cu at (279.4, 164.3)
- added MX76: MX-NoLED, MX_Only:MXOnly-1U-Hotswap-Antishear, F.Cu at (279.4, 183.4)
- added MX77: MX-NoLED, MX_Only:MXOnly-1U-Hotswap-Antishear, F.Cu at (279.4, 202.4)
- added MX78: MX-NoLED, MX_Only:MXOnly-1U-Hotswap-Antishear, F.Cu at (279.4, 221.5)
- added MX79: MX-NoLED, MX_Only:MXOnly-1U-Hotswap-Antishear, F.Cu at (298.4, 126.2)
- added MX8: MX-NoLED, MX_Only:MXOnly-1U-Hotswap-Antishear, F.Cu at (69.8, 145.3)
- added MX80: MX-NoLED, MX_Only:MXOnly-1U-Hotswap-Antishear, F.Cu at (298.4, 145.3)
- added MX81: MX-NoLED, MX_Only:MXOnly-1U-Hotswap-Antishear, F.Cu at (298.4, 164.3)
- added MX82: MX-NoLED, MX_Only:MXOnly-1U-Hotswap-Antishear, F.Cu at (298.4, 183.4)
- added MX83: MX-NoLED, MX_Only:MXOnly-1U-Hotswap-Antishear, F.Cu at (298.4, 202.4)
- added MX84: MX-NoLED, MX_Only:MXOnly-1U-Hotswap-Antishear, F.Cu at (298.4, 221.5)
- added MX85: MX-NoLED, MX_Only:MXOnly-1U-Hotswap-Antishear, F.Cu at (317.5, 126.2)
- added MX86: MX-NoLED, MX_Only:MXOnly-1U-Hotswap-Antishear, F.Cu at (317.5, 145.3)
- added MX87: MX-NoLED, MX_Only:MXOnly-1U-Hotswap-Antishear, F.Cu at (317.5, 164.3)
- added MX88: MX-NoLED, MX_Only:MXOnly-1U-Hotswap-Antishear, F.Cu at (317.5, 183.4)
- added MX89: MX-NoLED, MX_Only:MXOnly-1U-Hotswap-Antishear, F.Cu at (317.5, 202.4)
- added MX9: MX-NoLED, MX_Only:MXOnly-1U-Hotswap-Antishear, F.Cu at (69.8, 164.3)
- added MX90: MX-NoLED, MX_Only:MXOnly-1U-Hotswap-Antishear, F.Cu at (317.5, 221.5)
- added MX91: MX-NoLED, MX_Only:MXOnly-1U-Hotswap-Antishear, F.Cu at (336.6, 126.2)
- added MX92: MX-NoLED, MX_Only:MXOnly-1U-Hotswap-Antishear, F.Cu at (336.6, 145.3)
- added MX93: MX-NoLED, MX_Only:MXOnly-1U-Hotswap-Antishear, F.Cu at (336.6, 164.3)
- added MX94: MX-NoLED, MX_Only:MXOnly-1U-Hotswap-Antishear, F.Cu at (336.6, 183.4)
- added MX95: MX-NoLED, MX_Only:MXOnly-1U-Hotswap-Antishear, F.Cu at (336.6, 202.4)
- added MX96: MX-NoLED, MX_Only:MXOnly-1U-Hotswap-Antishear, F.Cu at (336.6, 221.5)
- added MX97: MX-NoLED, MX_Only:MXOnly-1U-Hotswap-Antishear, F.Cu at (355.6, 126.2)
- added MX98: MX-NoLED, MX_Only:MXOnly-1U-Hotswap-Antishear, F.Cu at (355.6, 145.3)
- added MX99: MX-NoLED, MX_Only:MXOnly-1U-Hotswap-Antishear, F.Cu at (355.6, 164.3)
- added Q1: S8050, Package_TO_SOT_SMD:SOT-23, B.Cu at (306.1, 88.1)
- added R3: 10k, Resistor_SMD:R_0603_1608Metric_Pad0.98x0.95mm_HandSolder, B.Cu at (323.9, 101.3)
- added R4: 1k, Resistor_SMD:R_0603_1608Metric_Pad0.98x0.95mm_HandSolder, B.Cu at (317.2, 90.3)
- added R5: 1k, Resistor_SMD:R_0603_1608Metric_Pad0.98x0.95mm_HandSolder, B.Cu at (327.2, 91.1)
- added R6: 1k, Resistor_SMD:R_0603_1608Metric_Pad0.98x0.95mm_HandSolder, B.Cu at (340.1, 91.0)
- added R7: 1k, Resistor_SMD:R_0603_1608Metric_Pad0.98x0.95mm_HandSolder, B.Cu at (303.1, 88.1)
- added SW1: RESET, acheron_Hardware:K2-1187SQ-A4SW-06, B.Cu at (319.8, 93.9)
- added U3: TPD4E05U06DQAR, acheron_Components:USON-10_2.5x1.0mm_P0.5mm, B.Cu at (356.1, 95.3)
- added Y1: 16Mhz, Crystal:Crystal_SMD_3225-4Pin_3.2x2.5mm_HandSoldering, B.Cu at (318.4, 100.3)
- D1, F1, J1, J2, L1, MH1, MH2, MH4, R1, R2: moved to B.Cu
- G1, G2: moved to F.Cu
- U1: value TPD4E05U06DQAR -> ATmega32U4-MU; footprint acheron_Components:USON-10_2.5x1.0mm_P0.5mm -> Package_DFN_QFN:QFN-44-1EP_7x7mm_P0.5mm_EP5.2x5.2mm; moved to B.Cu
- moved F1 296.8 mm to (363.2, 92.4)
- moved MH1 296.5 mm to (363.1, 87.8), turned to 180 degrees
- moved D1 295.3 mm to (362.5, 96.1), turned to 0 degrees
- moved R2 288.7 mm to (359.2, 96.4)
- moved G1 282.6 mm to (356.1, 95.7), turned to 0 degrees
- moved G2 282.6 mm to (356.1, 87.9), turned to 0 degrees
- moved J1 282.6 mm to (356.1, 94.1), turned to 0 degrees
- moved J2 282.6 mm to (356.1, 102.0), turned to 180 degrees
- moved R1 276.8 mm to (353.2, 96.4)
- moved L1 268.7 mm to (349.1, 95.1)
- moved MH2 268.7 mm to (349.1, 87.8), turned to 180 degrees
- moved MH4 268.7 mm to (349.1, 100.3), turned to 180 degrees
- moved U1 258.6 mm to (331.8, 96.9), turned to 180 degrees
Connections:
- J2 pad 4: GND -> GND1
- L1 pad 1: GND -> GND1
- U1 pad 1: DA+ -> ROW0
- U1 pad 10: DA+ -> ROW3
- U1 pad 2: DA- -> +VDC
- U1 pad 3: GNDPWR -> /MCU/DUSB+
- U1 pad 4: DA+ -> /MCU/DUSB-
- U1 pad 5: DA- -> GND
- U1 pad 6: DA- -> Net-(C7-Pad1)
- U1 pad 7: DA+ -> +VDC
- U1 pad 8: GNDPWR -> ROW1
- U1 pad 9: DA- -> ROW2
Routing:
- net ROW6: track 0.00 -> 536.4 mm
- net COL4: track 0.00 -> 508.4 mm, vias 0 -> 2
- net ROW7: track 0.00 -> 507.6 mm, vias 0 -> 2
- net COL5: track 0.00 -> 470.4 mm
- net ROW5: track 0.00 -> 445.7 mm, vias 0 -> 10
- net COL2: track 0.00 -> 432.4 mm, vias 0 -> 4
- net COL0: track 0.00 -> 432.1 mm
- net COL3: track 0.00 -> 430.0 mm, vias 0 -> 2
- net COL11: track 0.00 -> 427.8 mm, vias 0 -> 5
- net COL1: track 0.00 -> 422.0 mm, vias 0 -> 4
- net COL7: track 0.00 -> 418.0 mm, vias 0 -> 1
- net ROW4: track 0.00 -> 411.8 mm, vias 0 -> 8
- net COL6: track 0.00 -> 409.7 mm, vias 0 -> 1
- net COL8: track 0.00 -> 406.4 mm, vias 0 -> 2
- net COL10: track 0.00 -> 403.1 mm, vias 0 -> 6
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- added copper zone on B.Cu, net GND
- added copper zone on F.Cu, net GND
Other:
- board size 18 x 16.5 mm -> 323.9 x 145.3 mm
- net class Power: trace_width 0.508 -> 0.381
- board text added: "5V"
- board text added: "AREF"
- board text added: "B0"
- board text added: "B1"
- board text added: "B2"
- board text added: "B3"
- board text added: "B4"
- board text added: "B5"
- board text added: "B6"
- board text added: "B7"
- board text added: "C6"
- board text added: "C7"
- board text added: "CLK"
- board text added: "COL10"
- board text added: "COL12"
- board text added: "COL14"
- board text added: "COL4"
- board text added: "D0"
- board text added: "D1"
- board text added: "D2"
- board text added: "D3"
- board text added: "D4"
- board text added: "D5"
- board text added: "D6"
- board text added: "D7"
- board text added: "DT"
- board text added: "E2"
- board text added: "E6"
- board text added: "F0"
- board text added: "F1"
- board text added: "F4"
- board text added: "F5"
- board text added: "F6"
- board text added: "F7"
- board text added: "GND"
- board text added: "POTO REV2"
- board text added: "RGB"
- board text added: "ROW3"
- board text added: "ROW4"
- board text added: "ROW5"
- board text added: "RST"
- board text added: "SCL"
- board text added: "SDA"
- board text added: "SW"
