File: Poto-Rev2/Poto-Rev2.kicad_pcb (KiCad board)
At the start: 2 copper layers, 323.9 x 145.3 mm, 266 parts, among them J1 TYPE-C-31-M12_13, J10 Conn_01x01, J12 Conn_01x01, J15 OLED, J2 SM04B-SRSS-TB(LF)(SN), J3 Conn_01x12, J4 RGB, J5 ENCODER, J6 USB, J7 Conn_01x12, J8 Conn_01x01, J9 Conn_01x05, Q1 S8050, SW1 RESET, U1 ATmega32U4-MU, U3 TPD4E05U06DQAR, Y1 16Mhz

Commit message: uwu
awa
Parts:
- added J11: Conn_01x01, Connector_Wire:SolderWirePad_1x01_SMD_1x2mm, B.Cu at (347.3, 117.3)
- added J13: Conn_01x01, Connector_Wire:SolderWirePad_1x01_SMD_1x2mm, B.Cu at (327.8, 120.0)
- added J14: Conn_01x01, Connector_Wire:SolderWirePad_1x01_SMD_1x2mm, B.Cu at (309.2, 118.6)
- added J16: Conn_01x01, Connector_Wire:SolderWirePad_1x01_SMD_1x2mm, B.Cu at (291.6, 118.5)
- added J17: Conn_01x01, Connector_Wire:SolderWirePad_1x01_SMD_1x2mm, B.Cu at (287.7, 118.5)
- added J18: Conn_01x01, Connector_Wire:SolderWirePad_1x01_SMD_1x2mm, B.Cu at (254.0, 117.3)
- added J19: Conn_01x01, Connector_Wire:SolderWirePad_1x01_SMD_1x2mm, B.Cu at (249.6, 117.3)
- added J20: Conn_01x01, Connector_Wire:SolderWirePad_1x01_SMD_1x2mm, B.Cu at (230.5, 118.0)
- added J21: Conn_01x01, Connector_Wire:SolderWirePad_1x01_SMD_1x2mm, B.Cu at (211.3, 118.0)
- added J22: Conn_01x01, Connector_Wire:SolderWirePad_1x01_SMD_1x2mm, B.Cu at (192.4, 118.0)
- added J23: Conn_01x01, Connector_Wire:SolderWirePad_1x01_SMD_1x2mm, B.Cu at (173.2, 118.1)
- added J24: Conn_01x01, Connector_Wire:SolderWirePad_1x01_SMD_1x2mm, B.Cu at (154.2, 118.0)
- added J25: Conn_01x01, Connector_Wire:SolderWirePad_1x01_SMD_1x2mm, B.Cu at (135.1, 118.1)
- added J26: Conn_01x01, Connector_Wire:SolderWirePad_1x01_SMD_1x2mm, B.Cu at (359.8, 134.6)
- added J27: Conn_01x01, Connector_Wire:SolderWirePad_1x01_SMD_1x2mm, B.Cu at (360.0, 151.6)
- added J28: Conn_01x01, Connector_Wire:SolderWirePad_1x01_SMD_1x2mm, B.Cu at (359.9, 172.7)
- added J29: Conn_01x01, Connector_Wire:SolderWirePad_1x01_SMD_1x2mm, B.Cu at (360.4, 189.7)
- added J30: Conn_01x01, Connector_Wire:SolderWirePad_1x01_SMD_1x2mm, B.Cu at (359.8, 210.7)
- added J31: Conn_01x01, Connector_Wire:SolderWirePad_1x01_SMD_1x2mm, B.Cu at (360.4, 227.8)
- added J32: Conn_01x01, Connector_Wire:SolderWirePad_1x01_SMD_1x2mm, B.Cu at (78.7, 118.0)
- added J33: Conn_01x01, Connector_Wire:SolderWirePad_1x01_SMD_1x2mm, B.Cu at (116.8, 118.0)
- LED: renamed from LED2; footprint LED_SMD:LED_0201_0603Metric_Pad0.64x0.40mm_HandSolder -> LED_SMD:LED_0402_1005Metric_Pad0.77x0.64mm_HandSolder
- PWR: renamed from LED1; footprint LED_SMD:LED_0201_0603Metric_Pad0.64x0.40mm_HandSolder -> LED_SMD:LED_0402_1005Metric_Pad0.77x0.64mm_HandSolder
- moved LED 0.13 mm to (320.0, 90.6)
Routing:
- net COL1: track 422.0 -> 439.9 mm
- net COL6: track 409.7 -> 424.4 mm
- net COL5: track 470.4 -> 484.8 mm
- net COL3: track 430.0 -> 444.4 mm
- net COL4: track 508.4 -> 522.7 mm
- net COL2: track 432.4 -> 446.6 mm
- net COL0: track 432.1 -> 446.3 mm
- net COL12: track 203.3 -> 213.2 mm
- net COL7: track 418.0 -> 425.4 mm
- net COL10: track 403.1 -> 410.0 mm
- net COL8: track 406.4 -> 413.2 mm, vias 2 -> 3
- net COL11: track 427.8 -> 434.2 mm
- net COL9: track 402.9 -> 409.4 mm
- net ROW6: track 536.4 -> 539.7 mm
- net ROW7: track 507.6 -> 509.5 mm
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