File: Poto-Rev2/Poto-Rev2.sch (KiCad schematic (older format))
At the start: 0 parts

Commit message: Big Chungus Update
Almost Everything Done
Changed lines of the file:
@@
 $Descr A4 11693 8268
 encoding utf-8
-Sheet 1 2
+Sheet 1 4
 Title ""
 Date ""
@@
 F1 "USBC.sch" 50
 $EndSheet
+$Sheet
+S 3350 1350 1050 900
+U 617DACE9
+F0 "MCU" 50
+F1 "MCU.sch" 50
+$EndSheet
+$Sheet
+S 5150 1350 1050 900
+U 617DADC5
+F0 "Matrix" 50
+F1 "Matrix.sch" 50
+$EndSheet
 $EndSCHEMATC
