File: Poto-Rev2/MCU.sch (KiCad schematic (older format))
At the start: 27 parts, among them J10 Conn_01x01, J12 Conn_01x01, J15 OLED, J3 Conn_01x12, J4 RGB, J5 ENCODER, J6 USB, J7 Conn_01x12, J8 Conn_01x01, J9 Conn_01x05, SW1 RESET, U1 ATmega32U4-MU, Y1 16Mhz

Commit message: added some pads
added some pads for columns and rows
Parts:
- C1, C2, C3, C4, C7: LCSC Part No (none) -> C1525; Manufacturer (none) -> Samsung Electro-Mechanics; Manufacturer Part No (none) -> CL05B104KO5NNNC; Package (none) -> 0402
- C5, C6: LCSC Part No (none) -> C32949; Manufacturer (none) -> Samsung Electro-Mechanics; Manufacturer Part No (none) -> CL05C100JB5NNNC; Package (none) -> 0402
- C8: LCSC Part No (none) -> C52923; Manufacturer (none) -> Samsung Electro-Mechanics; Manufacturer Part No (none) -> CL05A105KA5NQNC; Package (none) -> 0402
- LED1, LED2: footprint LED_SMD:LED_0201_0603Metric_Pad0.64x0.40mm_HandSolder -> LED_SMD:LED_0603_1608Metric_Pad1.05x0.95mm_HandSolder
Changed lines of the file:
@@
 F 0 "LED1" V 2496 1280 50  0000 R CNN
 F 1 "PWR" V 2405 1280 50  0000 R CNN
-F 2 "LED_SMD:LED_0201_0603Metric_Pad0.64x0.40mm_HandSolder" V 2450 1350 50  0001 C CNN
+F 2 "LED_SMD:LED_0603_1608Metric_Pad1.05x0.95mm_HandSolder" V 2450 1350 50  0001 C CNN
 F 3 "~" V 2450 1350 50  0001 C CNN
 	1    2450 1350
@@
 F 2 "Capacitor_SMD:C_0402_1005Metric_Pad0.74x0.62mm_HandSolder" H 3200 1050 50  0001 C CNN
 F 3 "~" H 3200 1050 50  0001 C CNN
+F 4 "C1525" H 3200 1050 50  0001 C CNN "LCSC Part No"
+F 5 "Samsung Electro-Mechanics" H 3200 1050 50  0001 C CNN "Manufacturer"
+F 6 "CL05B104KO5NNNC" H 3200 1050 50  0001 C CNN "Manufacturer Part No"
+F 7 "0402" H 3200 1050 50  0001 C CNN "Package"
 	1    3200 1050
 	1    0    0    -1
@@
 F 2 "Capacitor_SMD:C_0402_1005Metric_Pad0.74x0.62mm_HandSolder" H 3600 1050 50  0001 C CNN
 F 3 "~" H 3600 1050 50  0001 C CNN
+F 4 "C1525" H 3600 1050 50  0001 C CNN "LCSC Part No"
+F 5 "Samsung Electro-Mechanics" H 3600 1050 50  0001 C CNN "Manufacturer"
+F 6 "CL05B104KO5NNNC" H 3600 1050 50  0001 C CNN "Manufacturer Part No"
+F 7 "0402" H 3600 1050 50  0001 C CNN "Package"
 	1    3600 1050
 	1    0    0    -1
@@
 F 2 "Capacitor_SMD:C_0402_1005Metric_Pad0.74x0.62mm_HandSolder" H 4000 1050 50  0001 C CNN
 F 3 "~" H 4000 1050 50  0001 C CNN
+F 4 "C1525" H 4000 1050 50  0001 C CNN "LCSC Part No"
+F 5 "Samsung Electro-Mechanics" H 4000 1050 50  0001 C CNN "Manufacturer"
+F 6 "CL05B104KO5NNNC" H 4000 1050 50  0001 C CNN "Manufacturer Part No"
+F 7 "0402" H 4000 1050 50  0001 C CNN "Package"
 	1    4000 1050
 	1    0    0    -1
@@
 F 2 "Capacitor_SMD:C_0402_1005Metric_Pad0.74x0.62mm_HandSolder" H 4400 1050 50  0001 C CNN
 F 3 "~" H 4400 1050 50  0001 C CNN
+F 4 "C1525" H 4400 1050 50  0001 C CNN "LCSC Part No"
+F 5 "Samsung Electro-Mechanics" H 4400 1050 50  0001 C CNN "Manufacturer"
+F 6 "CL05B104KO5NNNC" H 4400 1050 50  0001 C CNN "Manufacturer Part No"
+F 7 "0402" H 4400 1050 50  0001 C CNN "Package"
 	1    4400 1050
 	1    0    0    -1
@@
 F 0 "LED2" V 2146 2280 50  0000 R CNN
 F 1 "BuiltIn" V 2055 2280 50  0000 R CNN
-F 2 "LED_SMD:LED_0201_0603Metric_Pad0.64x0.40mm_HandSolder" V 2100 2350 50  0001 C CNN
+F 2 "LED_SMD:LED_0603_1608Metric_Pad1.05x0.95mm_HandSolder" V 2100 2350 50  0001 C CNN
 F 3 "~" V 2100 2350 50  0001 C CNN
 	1    2100 2350
@@
 F 2 "Capacitor_SMD:C_0402_1005Metric_Pad0.74x0.62mm_HandSolder" H 6000 2100 50  0001 C CNN
 F 3 "~" H 6000 2100 50  0001 C CNN
+F 4 "C32949" H 6000 2100 50  0001 C CNN "LCSC Part No"
+F 5 "Samsung Electro-Mechanics" H 6000 2100 50  0001 C CNN "Manufacturer"
+F 6 "CL05C100JB5NNNC" H 6000 2100 50  0001 C CNN "Manufacturer Part No"
+F 7 "0402" H 6000 2100 50  0001 C CNN "Package"
 	1    6000 2100
 	0    1    1    0
@@
 F 2 "Capacitor_SMD:C_0402_1005Metric_Pad0.74x0.62mm_HandSolder" H 6000 2700 50  0001 C CNN
 F 3 "~" H 6000 2700 50  0001 C CNN
+F 4 "C32949" H 6000 2700 50  0001 C CNN "LCSC Part No"
+F 5 "Samsung Electro-Mechanics" H 6000 2700 50  0001 C CNN "Manufacturer"
+F 6 "CL05C100JB5NNNC" H 6000 2700 50  0001 C CNN "Manufacturer Part No"
+F 7 "0402" H 6000 2700 50  0001 C CNN "Package"
 	1    6000 2700
 	0    1    1    0
@@
 F 2 "Capacitor_SMD:C_0402_1005Metric_Pad0.74x0.62mm_HandSolder" H 6900 3800 50  0001 C CNN
 F 3 "~" H 6900 3800 50  0001 C CNN
+F 4 "C1525" H 6900 3800 50  0001 C CNN "LCSC Part No"
+F 5 "Samsung Electro-Mechanics" H 6900 3800 50  0001 C CNN "Manufacturer"
+F 6 "CL05B104KO5NNNC" H 6900 3800 50  0001 C CNN "Manufacturer Part No"
+F 7 "0402" H 6900 3800 50  0001 C CNN "Package"
 	1    6900 3800
 	1    0    0    -1
@@
 F 2 "Capacitor_SMD:C_0402_1005Metric_Pad0.74x0.62mm_HandSolder" H 6250 3800 50  0001 C CNN
 F 3 "~" H 6250 3800 50  0001 C CNN
+F 4 "C52923" H 6250 3800 50  0001 C CNN "LCSC Part No"
+F 5 "Samsung Electro-Mechanics" H 6250 3800 50  0001 C CNN "Manufacturer"
+F 6 "CL05A105KA5NQNC" H 6250 3800 50  0001 C CNN "Manufacturer Part No"
+F 7 "0402" H 6250 3800 50  0001 C CNN "Package"
 	1    6250 3800
 	1    0    0    -1

Commit message: uwu
awa
Parts:
- C1, C2, C3, C4, C7: LCSC (none) -> C1525
- C5, C6: LCSC (none) -> C32949
- C8: LCSC (none) -> C52923
- LED1: footprint LED_SMD:LED_0603_1608Metric_Pad1.05x0.95mm_HandSolder -> LED_SMD:LED_0402_1005Metric_Pad0.77x0.64mm_HandSolder; LCSC (none) -> C130719; LCSC Part No (none) -> C130719; Manufacturer (none) -> Foshan NationStar Optoelectronics; Manufacturer Part No (none) -> NCD0402R1; Package (none) -> 0402
- LED2: footprint LED_SMD:LED_0603_1608Metric_Pad1.05x0.95mm_HandSolder -> LED_SMD:LED_0402_1005Metric_Pad0.77x0.64mm_HandSolder; LCSC (none) -> C397046; LCSC Part No (none) -> C397046; Manufacturer (none) -> MEIHUA; Manufacturer Part No (none) -> MHT136WDT-C2; Package (none) -> 0402
- R3: LCSC (none) -> C25804; LCSC Part No (none) -> C25804
- R4, R5, R6: LCSC (none) -> C21190; LCSC Part No (none) -> C21190
- SW1: LCSC (none) -> C92584; LCSC Part No (none) -> C92584; Manufacturer (none) -> Korean Hroparts Elec; Manufacturer Part No (none) -> K2-1187SQ-A4SW-06; Package (none) -> SW-SMD-4_5.2x5.2x3.7P
- U1: LCSC (none) -> C112161; LCSC Part No (none) -> C112161
- Y1: LCSC (none) -> C13738; LCSC Part No (none) -> C13738
Changed lines of the file:
@@
 F 2 "acheron_Hardware:K2-1187SQ-A4SW-06" H 1050 1400 50  0001 C CNN
 F 3 "~" H 1050 1400 50  0001 C CNN
+F 4 "C92584" H 1050 1200 50  0001 C CNN "LCSC Part No"
+F 5 "Korean Hroparts Elec" H 1050 1200 50  0001 C CNN "Manufacturer"
+F 6 "K2-1187SQ-A4SW-06" H 1050 1200 50  0001 C CNN "Manufacturer Part No"
+F 7 "SW-SMD-4_5.2x5.2x3.7P" H 1050 1200 50  0001 C CNN "Package"
+F 8 "C92584" H 1050 1200 50  0001 C CNN "LCSC"
 	1    1050 1200
 	1    0    0    -1
@@
 F 2 "Resistor_SMD:R_0603_1608Metric_Pad0.98x0.95mm_HandSolder" H 1500 1050 50  0001 C CNN
 F 3 "~" H 1500 1050 50  0001 C CNN
+F 4 "C25804" H 1500 1050 50  0001 C CNN "LCSC Part No"
+F 5 "C25804" H 1500 1050 50  0001 C CNN "LCSC"
 	1    1500 1050
 	1    0    0    -1
@@
 F 2 "Resistor_SMD:R_0603_1608Metric_Pad0.98x0.95mm_HandSolder" H 1900 1050 50  0001 C CNN
 F 3 "~" H 1900 1050 50  0001 C CNN
+F 4 "C21190" H 1900 1050 50  0001 C CNN "LCSC Part No"
+F 5 "C21190" H 1900 1050 50  0001 C CNN "LCSC"
 	1    1900 1050
 	1    0    0    -1
@@
 F 2 "Resistor_SMD:R_0603_1608Metric_Pad0.98x0.95mm_HandSolder" H 2450 1050 50  0001 C CNN
 F 3 "~" H 2450 1050 50  0001 C CNN
+F 4 "C21190" H 2450 1050 50  0001 C CNN "LCSC Part No"
+F 5 "C21190" H 2450 1050 50  0001 C CNN "LCSC"
 	1    2450 1050
 	1    0    0    -1
@@
 F 0 "LED1" V 2496 1280 50  0000 R CNN
 F 1 "PWR" V 2405 1280 50  0000 R CNN
-F 2 "LED_SMD:LED_0603_1608Metric_Pad1.05x0.95mm_HandSolder" V 2450 1350 50  0001 C CNN
+F 2 "LED_SMD:LED_0402_1005Metric_Pad0.77x0.64mm_HandSolder" V 2450 1350 50  0001 C CNN
 F 3 "~" V 2450 1350 50  0001 C CNN
+F 4 "C130719" H 2450 1350 50  0001 C CNN "LCSC Part No"
+F 5 "NCD0402R1" H 2450 1350 50  0001 C CNN "Manufacturer Part No"
+F 6 "Foshan NationStar Optoelectronics" H 2450 1350 50  0001 C CNN "Manufacturer"
+F 7 "0402" H 2450 1350 50  0001 C CNN "Package"
+F 8 "C130719" H 2450 1350 50  0001 C CNN "LCSC"
 	1    2450 1350
 	0    -1   -1   0
@@
 F 6 "CL05B104KO5NNNC" H 3200 1050 50  0001 C CNN "Manufacturer Part No"
 F 7 "0402" H 3200 1050 50  0001 C CNN "Package"
+F 8 "C1525" H 3200 1050 50  0001 C CNN "LCSC"
 	1    3200 1050
 	1    0    0    -1
@@
 F 6 "CL05B104KO5NNNC" H 3600 1050 50  0001 C CNN "Manufacturer Part No"
 F 7 "0402" H 3600 1050 50  0001 C CNN "Package"
+F 8 "C1525" H 3600 1050 50  0001 C CNN "LCSC"
 	1    3600 1050
 	1    0    0    -1
@@
 F 6 "CL05B104KO5NNNC" H 4000 1050 50  0001 C CNN "Manufacturer Part No"
 F 7 "0402" H 4000 1050 50  0001 C CNN "Package"
+F 8 "C1525" H 4000 1050 50  0001 C CNN "LCSC"
 	1    4000 1050
 	1    0    0    -1
@@
 F 6 "CL05B104KO5NNNC" H 4400 1050 50  0001 C CNN "Manufacturer Part No"
 F 7 "0402" H 4400 1050 50  0001 C CNN "Package"
+F 8 "C1525" H 4400 1050 50  0001 C CNN "LCSC"
 	1    4400 1050
 	1    0    0    -1
@@
 F 2 "Resistor_SMD:R_0603_1608Metric_Pad0.98x0.95mm_HandSolder" H 1850 2150 50  0001 C CNN
 F 3 "~" H 1850 2150 50  0001 C CNN
+F 4 "C21190" H 1850 2150 50  0001 C CNN "LCSC Part No"
+F 5 "C21190" H 1850 2150 50  0001 C CNN "LCSC"
 	1    1850 2150
 	0    1    1    0
@@
 F 0 "LED2" V 2146 2280 50  0000 R CNN
 F 1 "BuiltIn" V 2055 2280 50  0000 R CNN
-F 2 "LED_SMD:LED_0603_1608Metric_Pad1.05x0.95mm_HandSolder" V 2100 2350 50  0001 C CNN
+F 2 "LED_SMD:LED_0402_1005Metric_Pad0.77x0.64mm_HandSolder" V 2100 2350 50  0001 C CNN
 F 3 "~" V 2100 2350 50  0001 C CNN
+F 4 "C397046" H 2100 2350 50  0001 C CNN "LCSC Part No"
+F 5 "MEIHUA" H 2100 2350 50  0001 C CNN "Manufacturer"
+F 6 "MHT136WDT-C2" H 2100 2350 50  0001 C CNN "Manufacturer Part No"
+F 7 "0402" H 2100 2350 50  0001 C CNN "Package"
+F 8 "C397046" H 2100 2350 50  0001 C CNN "LCSC"
 	1    2100 2350
 	0    -1   -1   0
@@
 F 2 "Package_DFN_QFN:QFN-44-1EP_7x7mm_P0.5mm_EP5.2x5.2mm" H 8250 3600 50  0001 C CIN
 F 3 "http://ww1.microchip.com/downloads/en/DeviceDoc/Atmel-7766-8-bit-AVR-ATmega16U4-32U4_Datasheet.pdf" H 8250 3600 50  0001 C CNN
+F 4 "C112161" H 8250 3600 50  0001 C CNN "LCSC Part No"
+F 5 "C112161" H 8250 3600 50  0001 C CNN "LCSC"
 	1    8250 3600
 	1    0    0    -1
@@
 F 2 "Crystal:Crystal_SMD_3225-4Pin_3.2x2.5mm_HandSoldering" H 6400 2400 50  0001 C CNN
 F 3 "~" H 6400 2400 50  0001 C CNN
+F 4 "C13738" H 6400 2400 50  0001 C CNN "LCSC Part No"
+F 5 "C13738" H 6400 2400 50  0001 C CNN "LCSC"
 	1    6400 2400
 	0    1    1    0
@@
 F 6 "CL05C100JB5NNNC" H 6000 2100 50  0001 C CNN "Manufacturer Part No"
 F 7 "0402" H 6000 2100 50  0001 C CNN "Package"
+F 8 "C32949" H 6000 2100 50  0001 C CNN "LCSC"
 	1    6000 2100
 	0    1    1    0
@@
 F 6 "CL05C100JB5NNNC" H 6000 2700 50  0001 C CNN "Manufacturer Part No"
 F 7 "0402" H 6000 2700 50  0001 C CNN "Package"
+F 8 "C32949" H 6000 2700 50  0001 C CNN "LCSC"
 	1    6000 2700
 	0    1    1    0
@@
 F 6 "CL05B104KO5NNNC" H 6900 3800 50  0001 C CNN "Manufacturer Part No"
 F 7 "0402" H 6900 3800 50  0001 C CNN "Package"
+F 8 "C1525" H 6900 3800 50  0001 C CNN "LCSC"
 	1    6900 3800
 	1    0    0    -1
@@
 F 6 "CL05A105KA5NQNC" H 6250 3800 50  0001 C CNN "Manufacturer Part No"
 F 7 "0402" H 6250 3800 50  0001 C CNN "Package"
+F 8 "C52923" H 6250 3800 50  0001 C CNN "LCSC"
 	1    6250 3800
 	1    0    0    -1
