File: Poto-Rev2/Matrix.sch (KiCad schematic (older format))
At the start: 206 parts, among them Q1 S8050

Commit message: uwu
awa
Parts:
- added J11, J13, J14, J16, J17, J18, J19, J20, J21, J22, J23, J24, J25, J26, J27, J28, J29, J30, J31, J32, J33: Conn_01x01, Connector_Wire:SolderWirePad_1x01_SMD_1x2mm, symbol Connector_Generic:Conn_01x01
- D10, D100, D101, D102, D103, D11, D12, D13, D14, D15, D16, D17, D18, D19, D2, D20, D21, D22, D23, D24, D25, D26, D27, D28, D29, D3, D30, D31, D32, D33, D34, D35, D36, D37, D38, D39, D4, D40, D41, D42, D43, D44, D45, D46, D47, D48, D49, D5, D50, D51, D52, D53, D54, D55, D56, D57, D58, D59, D6, D60, D61, D62, D63, D64, D65, D66, D67, D68, D69, D7, D70, D71, D72, D73, D74, D75, D76, D77, D78, D79, D8, D80, D81, D82, D83, D84, D85, D86, D87, D88, D89, D9, D90, D91, D92, D93, D94, D95, D96, D97, D98, D99: LCSC (none) -> C81598; LCSC Part No (none) -> C81598
- Q1: LCSC (none) -> C2150; LCSC Part No (none) -> C2150; Manufacturer (none) -> Changjiang Electronics Tech (CJ); Manufacturer Part No (none) -> SS8050; Package (none) -> SOT-23-3
- R7: LCSC (none) -> C21190; LCSC Part No (none) -> C21190
Connections:
- net COL0: now also J25.1 (Pin_1)
- net COL1: now also J24.1 (Pin_1)
- net COL10: now also J14.1 (Pin_1)
- net COL11: now also J13.1 (Pin_1)
- net COL12: now also J11.1 (Pin_1)
- net COL2: now also J23.1 (Pin_1)
- net COL3: now also J22.1 (Pin_1)
- net COL4: now also J21.1 (Pin_1)
- net COL5: now also J20.1 (Pin_1)
- net COL6: now also J19.1 (Pin_1)
- net COL7: now also J18.1 (Pin_1)
- net COL8: now also J17.1 (Pin_1)
- net COL9: now also J16.1 (Pin_1)
- net ROW0: now also J26.1 (Pin_1)
- net ROW1: now also J27.1 (Pin_1)
- net ROW2: now also J28.1 (Pin_1)
- net ROW3: now also J29.1 (Pin_1)
- net ROW4: now also J30.1 (Pin_1)
- net ROW5: now also J31.1 (Pin_1)
- net ROW6: now also J32.1 (Pin_1)
- net ROW7: now also J33.1 (Pin_1)
