File: Poto-Rev2/USBC.sch (KiCad schematic (older format))
At the start: 14 parts, among them J1 TYPE-C-31-M12_13, J2 SM04B-SRSS-TB(LF)(SN), U1 TPD4E05U06DQAR

Commit message: fixing libraries and setting up stuff
Parts:
- R1, R2: footprint Resistors_SMD:R_0603 -> Resistor_SMD:R_0603_1608Metric
Changed lines of the file:
@@
 F 0 "R1" V 2400 1675 30  0000 C CNN
 F 1 "5.1k" V 2325 1675 30  0000 C CNN
-F 2 "Resistors_SMD:R_0603" H 2325 1675 50  0001 C CNN
+F 2 "Resistor_SMD:R_0603_1608Metric" H 2325 1675 50  0001 C CNN
 F 3 "~" H 2325 1675 50  0001 C CNN
 F 4 "R0603" V 2325 1675 50  0001 C CNN "Package"
@@
 F 0 "R2" V 2400 1875 30  0000 C CNN
 F 1 "5.1k" V 2325 1875 30  0000 C CNN
-F 2 "Resistors_SMD:R_0603" H 2325 1875 50  0001 C CNN
+F 2 "Resistor_SMD:R_0603_1608Metric" H 2325 1875 50  0001 C CNN
 F 3 "~" H 2325 1875 50  0001 C CNN
 F 4 "R0603" V 2325 1875 50  0001 C CNN "Package"
@@
 U 1 1 5C91EC0E
 P 6950 1625
+AR Path="/5C91EC0E" Ref="MH1"  Part="1"
+AR Path="/6159038F/5C91EC0E" Ref="MH1"  Part="1"
 F 0 "MH1" H 7029 1667 50  0000 L CNN
 F 1 "Mount-M2" H 7029 1576 50  0000 L CNN
@@
 U 1 1 5C91EC94
 P 6950 1800
+AR Path="/5C91EC94" Ref="MH2"  Part="1"
+AR Path="/6159038F/5C91EC94" Ref="MH2"  Part="1"
 F 0 "MH2" H 7029 1842 50  0000 L CNN
 F 1 "Mount-M2" H 7029 1751 50  0000 L CNN
@@
 U 1 1 5C91ECC0
 P 6950 1975
+AR Path="/5C91ECC0" Ref="MH3"  Part="1"
+AR Path="/6159038F/5C91ECC0" Ref="MH3"  Part="1"
 F 0 "MH3" H 7029 2017 50  0000 L CNN
 F 1 "Mount-M2" H 7029 1926 50  0000 L CNN
@@
 U 1 1 5C91ECE4
 P 6950 2150
+AR Path="/5C91ECE4" Ref="MH4"  Part="1"
+AR Path="/6159038F/5C91ECE4" Ref="MH4"  Part="1"
 F 0 "MH4" H 7029 2192 50  0000 L CNN
 F 1 "Mount-M2" H 7029 2101 50  0000 L CNN
@@
 U 1 1 5E787D68
 P 4375 1725
+AR Path="/5E787D68" Ref="U1"  Part="1"
+AR Path="/6159038F/5E787D68" Ref="U1"  Part="1"
 F 0 "U1" H 4375 2191 50  0000 C CNN
 F 1 "TPD4E05U06DQAR" H 4375 2100 50  0000 C CNN

Commit message: Big Chungus Update
Almost Everything Done
Parts:
- J1: symbol acheronSymbols:TYPE-C-31-M12_13-acheronSymbols -> acheronSymbols:TYPE-C-31-M12_13
- U1: symbol acheronSymbols:TPD4E05U06DQAR-acheronSymbols -> acheronSymbols:TPD4E05U06DQAR
Connections:
- net GND renamed GND1
Changed lines of the file:
@@
 $Descr A4 11693 8268
 encoding utf-8
-Sheet 2 2
+Sheet 2 4
 Title ""
 Date ""
@@
 $EndComp
 $Comp
-L power:GND #PWR0109
-U 1 1 5E792568
-P 1275 4350
-F 0 "#PWR0109" H 1275 4100 50  0001 C CNN
-F 1 "GND" H 1275 4225 20  0000 C CNN
-F 2 "" H 1275 4350 50  0001 C CNN
-F 3 "" H 1275 4350 50  0001 C CNN
-	1    1275 4350
-	-1   0    0    1
-$EndComp
-$Comp
-L power:GND #PWR0104
-U 1 1 5C91E0CE
-P 9225 3250
-F 0 "#PWR0104" H 9225 3000 50  0001 C CNN
-F 1 "GND" H 9230 3077 50  0000 C CNN
-F 2 "" H 9225 3250 50  0001 C CNN
-F 3 "" H 9225 3250 50  0001 C CNN
-	1    9225 3250
-	1    0    0    -1
-$EndComp
-$Comp
 L Device:R_Small R1
 U 1 1 5C91B042
@@
 U 1 1 5E18209E
 P 4475 3550
+AR Path="/5E18209E" Ref="D1"  Part="1"
+AR Path="/6159038F/5E18209E" Ref="D1"  Part="1"
 F 0 "D1" H 4475 3400 30  0000 C CNN
 F 1 "SMF9.0CA" H 4475 3450 30  0000 C CNN
@@
 $EndComp
 $Comp
-L acheronSymbols:TPD4E05U06DQAR-acheronSymbols U1
+L acheronSymbols:TPD4E05U06DQAR U1
 U 1 1 5E787D68
 P 4375 1725
 AR Path="/5E787D68" Ref="U1"  Part="1"
-AR Path="/6159038F/5E787D68" Ref="U1"  Part="1"
-F 0 "U1" H 4375 2191 50  0000 C CNN
+AR Path="/6159038F/5E787D68" Ref="U3"  Part="1"
+F 0 "U3" H 4375 2191 50  0000 C CNN
 F 1 "TPD4E05U06DQAR" H 4375 2100 50  0000 C CNN
 F 2 "acheron_Components:USON-10_2.5x1.0mm_P0.5mm" H 4375 2775 50  0001 C CNN
@@
 $EndComp
 $Comp
-L acheronSymbols:TYPE-C-31-M12_13-acheronSymbols J1
+L acheronSymbols:TYPE-C-31-M12_13 J1
 U 1 1 5E77A5D1
 P 1575 2325
+AR Path="/5E77A5D1" Ref="J1"  Part="1"
+AR Path="/6159038F/5E77A5D1" Ref="J1"  Part="1"
 F 0 "J1" H 1575 3750 50  0000 C CNN
 F 1 "TYPE-C-31-M12_13" H 1575 3650 50  0000 C CNN
@@
 	1    0    0    -1
 $EndComp
+$Comp
+L power:GND1 #PWR0104
+U 1 1 61F66A71
+P 1275 4350
+F 0 "#PWR0104" H 1275 4100 50  0001 C CNN
+F 1 "GND1" H 1280 4177 50  0000 C CNN
+F 2 "" H 1275 4350 50  0001 C CNN
+F 3 "" H 1275 4350 50  0001 C CNN
+	1    1275 4350
+	-1   0    0    1
+$EndComp
+$Comp
+L power:GND1 #PWR0109
+U 1 1 61F69EB7
+P 9225 3250
+F 0 "#PWR0109" H 9225 3000 50  0001 C CNN
+F 1 "GND1" H 9230 3077 50  0000 C CNN
+F 2 "" H 9225 3250 50  0001 C CNN
+F 3 "" H 9225 3250 50  0001 C CNN
+	1    9225 3250
+	1    0    0    -1
+$EndComp

Commit message: uwu
awa
Parts:
- D1: LCSC (none) -> C123799
- F1: LCSC (none) -> C135342
- J1: LCSC (none) -> C165948
- J2: LCSC (none) -> C160404
- L1: LCSC (none) -> C33600
- R1, R2: LCSC (none) -> C23186; LCSC Part No (none) -> C23186
- U1: LCSC (none) -> C138714
Changed lines of the file:
@@
 F 3 "~" H 2325 1675 50  0001 C CNN
 F 4 "R0603" V 2325 1675 50  0001 C CNN "Package"
+F 5 "C23186" H 2325 1675 50  0001 C CNN "LCSC Part No"
+F 6 "C23186" H 2325 1675 50  0001 C CNN "LCSC"
 	1    2325 1675
 	0    -1   -1   0
@@
 F 3 "~" H 2325 1875 50  0001 C CNN
 F 4 "R0603" V 2325 1875 50  0001 C CNN "Package"
+F 5 "C23186" H 2325 1875 50  0001 C CNN "LCSC Part No"
+F 6 "C23186" H 2325 1875 50  0001 C CNN "LCSC"
 	1    2325 1875
 	0    -1   -1   0
@@
 F 6 "C33600" H 1275 4525 50  0001 C CNN "LCSC Part No"
 F 7 "L1206" H 1275 4525 50  0001 C CNN "Package"
+F 8 "C33600" H 1275 4525 50  0001 C CNN "LCSC"
 	1    1275 4525
 	1    0    0    -1
@@
 F 6 "SMF9.0CA" H 4475 3550 50  0001 C CNN "Manufacturer Part No"
 F 7 "C123799" H 4475 3550 50  0001 C CNN "LCSC Part No"
+F 8 "C123799" H 4475 3550 50  0001 C CNN "LCSC"
 	1    4475 3550
 	0    1    -1   0
@@
 F 6 "C135342" V 4225 3350 50  0001 C CNN "LCSC Part No"
 F 7 "F1206" V 4225 3350 50  0001 C CNN "Package"
+F 8 "C135342" H 4225 3350 50  0001 C CNN "LCSC"
 	1    4225 3350
 	0    -1   -1   0
@@
 F 5 "SM04B-SRSS-TB(LF)(SN)" H 9500 3050 50  0001 C CNN "Manufacturer Part No"
 F 6 "C160404" H 9500 3050 50  0001 C CNN "LCSC Part No"
+F 7 "C160404" H 9500 3050 50  0001 C CNN "LCSC"
 	1    9500 3050
 	1    0    0    -1
@@
 F 6 "C138714" H 4375 2475 50  0001 C CNN "LCSC Part No"
 F 7 "uSON-10" H 4375 2575 50  0001 C CNN "Package"
+F 8 "C138714" H 4375 1725 50  0001 C CNN "LCSC"
 	1    4375 1725
 	1    0    0    -1
@@
 F 5 "TYPE-C-31-M-12" H 1575 2325 50  0001 C CNN "Manufacturer Part No"
 F 6 "C165948" H 1575 2325 50  0001 C CNN "LCSC Part No"
+F 7 "C165948" H 1575 2325 50  0001 C CNN "LCSC"
 	1    1575 2325
 	1    0    0    -1
